File: firstpcb.sch (KiCad schematic (older format))
At the start: 14 parts

Commit message: Renaming footprints
Parts:
- added D1, D2, D3, D4: SOD-123, Diode_SMD:D_SOD-123, symbol Device:D_Small
- added F1: 500mA, Fuse:Fuse_1206_3216Metric, symbol Device:Polyfuse
- added MX1, MX2, MX3, MX4: MX-NoLED, MX_Alps_Hybrid:MX-8U-NoLED, symbol MX_Alps_Hybrid:MX-NoLED
- added USB1: Molex-0548190589, random-keyboard-parts:Molex-0548190589, symbol random-keyboard-parts:Molex-0548190589
- C1, C2, C3, C4, C5, C6, C7: renamed from C?; footprint (none) -> Capacitor_SMD:C_0805_2012Metric
- R1, R2, R3, R4: renamed from R?; footprint (none) -> Resistor_SMD:R_0805_2012Metric
- SW1: renamed from SW?; footprint (none) -> random-keyboard-parts:SKQG-1155865
- Y1: renamed from Y?; footprint (none) -> Crystal:Crystal_SMD_3225-4Pin_3.2x2.5mm
- gave numbers to parts that had none: 1
Connections:
- net +5V: now also F1.1
- net D+: now also USB1.3 (D+)
- net D-: now also USB1.4 (D-)
- net GND: now also USB1.1 (GND)
- new net: D1.2 (A), MX1.2 (ROW)
- new net: D3.2 (A), MX3.2 (ROW)
- new net: D2.2 (A), MX2.2 (ROW)
- new net: D4.2 (A), MX4.2 (ROW)
- new net COL0: MX1.1 (COL), MX2.1 (COL)
- new net COL1: MX3.1 (COL), MX4.1 (COL)
- new net ROW0: D1.1 (K), D3.1 (K)
- new net ROW1: D2.1 (K), D4.1 (K)
- new net VCC: F1.2, USB1.5 (VBUS)

Commit message: First pcb export nothing changed yet
Parts:
- MX1, MX4: footprint MX_Alps_Hybrid:MX-8U-NoLED -> MX_Alps_Hybrid:MX-1U
- MX2: renamed from MX3; footprint MX_Alps_Hybrid:MX-8U-NoLED -> MX_Alps_Hybrid:MX-1U
- MX3: renamed from MX2; footprint MX_Alps_Hybrid:MX-8U-NoLED -> MX_Alps_Hybrid:MX-1U
- renumbered C3 to C1, C4 to C2, C6 to C3, C1 to C4, C2 to C5, C5 to C6, R3 to R1, R1 to R3
Connections:
- net COL0: now also U1.29 (PB5)
- net COL1: now also U1.28 (PB4)
- net GND: now also C2.1, U1.16 (XTAL2), Y1.3
- net ROW0: now also U1.27 (PD7)
- net ROW1: now also U1.30 (PB6)
Other:
- moved on the sheet: C1
Changed lines of the file:
@@
 EESchema Schematic File Version 4
+LIBS:firstpcb-cache
 EELAYER 30 0
 EELAYER END
@@
 Wire Wire Line
 	3900 2400 3900 2250
-Wire Wire Line
-	4100 2400 4000 2400
-Wire Wire Line
-	4000 2400 3900 2400
-Connection ~ 4000 2400
-Connection ~ 3900 2400
 $Comp
 L power:GND #PWR0102
@@
 $EndComp
 Wire Wire Line
-	4000 6000 3900 6000
-Connection ~ 3900 6000
-Wire Wire Line
 	3500 6000 3900 6000
 $Comp
@@
 $EndComp
 $Comp
-L Device:R_Small R1
+L Device:R_Small R3
 U 1 1 633F12B6
 P 2800 3800
-F 0 "R1" V 2604 3800 50  0000 C CNN
+F 0 "R3" V 2604 3800 50  0000 C CNN
 F 1 "22" V 2695 3800 50  0000 C CNN
 F 2 "Resistor_SMD:R_0805_2012Metric" H 2800 3800 50  0001 C CNN
@@
 	3000 3700 2550 3700
 $Comp
-L Device:C_Small C6
+L Device:C_Small C3
 U 1 1 633F29F6
 P 2950 4100
-F 0 "C6" H 3042 4146 50  0000 L CNN
+F 0 "C3" H 3042 4146 50  0000 L CNN
 F 1 "1uF" H 3042 4055 50  0000 L CNN
 F 2 "Capacitor_SMD:C_0805_2012Metric" H 2950 4100 50  0001 C CNN
@@
 $EndComp
 $Comp
-L Device:C_Small C5
+L Device:C_Small C6
 U 1 1 63405601
 P 2700 4850
-F 0 "C5" H 2792 4896 50  0000 L CNN
+F 0 "C6" H 2792 4896 50  0000 L CNN
 F 1 "0.1uF" H 2792 4805 50  0000 L CNN
 F 2 "Capacitor_SMD:C_0805_2012Metric" H 2700 4850 50  0001 C CNN
@@
 $EndComp
 $Comp
-L Device:C_Small C2
+L Device:C_Small C5
 U 1 1 63406236
 P 2300 4850
-F 0 "C2" H 2392 4896 50  0000 L CNN
+F 0 "C5" H 2392 4896 50  0000 L CNN
 F 1 "0.1uF" H 2392 4805 50  0000 L CNN
 F 2 "Capacitor_SMD:C_0805_2012Metric" H 2300 4850 50  0001 C CNN
@@
 $EndComp
 $Comp
-L Device:C_Small C1
+L Device:C_Small C4
 U 1 1 63406D59
 P 1900 4850
-F 0 "C1" H 1992 4896 50  0000 L CNN
+F 0 "C4" H 1992 4896 50  0000 L CNN
 F 1 "0.1uF" H 1992 4805 50  0000 L CNN
 F 2 "Capacitor_SMD:C_0805_2012Metric" H 1900 4850 50  0001 C CNN
@@
 	3400 2900 2900 2900
 $Comp
-L Device:C_Small C3
+L Device:C_Small C1
 U 1 1 634150DE
-P 2550 2800
-F 0 "C3" V 2321 2800 50  0000 C CNN
-F 1 "22pF" V 2412 2800 50  0000 C CNN
-F 2 "Capacitor_SMD:C_0805_2012Metric" H 2550 2800 50  0001 C CNN
-F 3 "~" H 2550 2800 50  0001 C CNN
-	1    2550 2800
-	0    1    1    0
-$EndComp
-$Comp
-L Device:C_Small C4
+P 2550 2750
+F 0 "C1" V 2321 2750 50  0000 C CNN
+F 1 "22pF" V 2412 2750 50  0000 C CNN
+F 2 "Capacitor_SMD:C_0805_2012Metric" H 2550 2750 50  0001 C CNN
+F 3 "~" H 2550 2750 50  0001 C CNN
+	1    2550 2750
+	0    1    1    0
+$EndComp
+$Comp
+L Device:C_Small C2
 U 1 1 6341688C
 P 2550 3200
-F 0 "C4" V 2321 3200 50  0000 C CNN
+F 0 "C2" V 2321 3200 50  0000 C CNN
 F 1 "22pF" V 2412 3200 50  0000 C CNN
 F 2 "Capacitor_SMD:C_0805_2012Metric" H 2550 3200 50  0001 C CNN
@@
 	0    1    1    0
 $EndComp
-Wire Wire Line
-	2900 2900 2650 2900
-Wire Wire Line
-	2650 2900 2650 2800
-Connection ~ 2900 2900
-Wire Wire Line
-	2450 2800 2450 3200
 Wire Wire Line
 	2650 3200 2650 3100
@@
 $EndComp
 Wire Wire Line
-	2450 3200 2450 3300
-Connection ~ 2450 3200
-Wire Wire Line
-	2800 3000 2800 3100
-Wire Wire Line
-	2800 3100 2800 3300
-Wire Wire Line
-	2800 3300 2450 3300
-Connection ~ 2450 3300
-Wire Wire Line
 	3000 3000 3050 3000
-Wire Wire Line
-	3050 3000 3050 3100
-Wire Wire Line
-	3050 3100 3050 3300
-Wire Wire Line
-	3050 3300 2800 3300
-Connection ~ 2800 3300
-Wire Wire Line
-	2650 3100 2900 3100
-Wire Wire Line
-	2900 3100 3400 3100
 $Comp
 L Switch:SW_Push SW1
@@
 	3300 2700 3350 2700
 $Comp
-L Device:R_Small R3
+L Device:R_Small R1
 U 1 1 6342361B
 P 3350 2350
-F 0 "R3" H 3409 2396 50  0000 L CNN
+F 0 "R1" H 3409 2396 50  0000 L CNN
 F 1 "10k" H 3409 2305 50  0000 L CNN
 F 2 "Resistor_SMD:R_0805_2012Metric" H 3350 2350 50  0001 C CNN
@@
 F 0 "MX1" H 8383 3323 60  0000 C CNN
 F 1 "MX-NoLED" H 8383 3249 20  0000 C CNN
-F 2 "MX_Alps_Hybrid:MX-8U-NoLED" H 7725 3075 60  0001 C CNN
+F 2 "MX_Alps_Hybrid:MX-1U" H 7725 3075 60  0001 C CNN
 F 3 "" H 7725 3075 60  0001 C CNN
 	1    8350 3100
@@
 	8150 3250 8300 3250
 $Comp
-L MX_Alps_Hybrid:MX-NoLED MX3
+L MX_Alps_Hybrid:MX-NoLED MX2
 U 1 1 63440E49
 P 9350 3100
-F 0 "MX3" H 9383 3323 60  0000 C CNN
+F 0 "MX2" H 9383 3323 60  0000 C CNN
 F 1 "MX-NoLED" H 9383 3249 20  0000 C CNN
-F 2 "MX_Alps_Hybrid:MX-8U-NoLED" H 8725 3075 60  0001 C CNN
+F 2 "MX_Alps_Hybrid:MX-1U" H 8725 3075 60  0001 C CNN
 F 3 "" H 8725 3075 60  0001 C CNN
 	1    9350 3100
@@
 	9150 3250 9300 3250
 $Comp
-L MX_Alps_Hybrid:MX-NoLED MX2
+L MX_Alps_Hybrid:MX-NoLED MX3
 U 1 1 63442A22
 P 8350 3800
-F 0 "MX2" H 8383 4023 60  0000 C CNN
+F 0 "MX3" H 8383 4023 60  0000 C CNN
 F 1 "MX-NoLED" H 8383 3949 20  0000 C CNN
-F 2 "MX_Alps_Hybrid:MX-8U-NoLED" H 7725 3775 60  0001 C CNN
+F 2 "MX_Alps_Hybrid:MX-1U" H 7725 3775 60  0001 C CNN
 F 3 "" H 7725 3775 60  0001 C CNN
 	1    8350 3800
@@
 F 0 "MX4" H 9383 4023 60  0000 C CNN
 F 1 "MX-NoLED" H 9383 3949 20  0000 C CNN
-F 2 "MX_Alps_Hybrid:MX-8U-NoLED" H 8725 3775 60  0001 C CNN
+F 2 "MX_Alps_Hybrid:MX-1U" H 8725 3775 60  0001 C CNN
 F 3 "" H 8725 3775 60  0001 C CNN
 	1    9350 3800
@@
 Text GLabel 9500 2700 1    50   Input ~ 0
 COL1
+Wire Wire Line
+	3900 2400 4000 2400
+Connection ~ 3900 2400
+Text GLabel 4600 4600 2    50   Input ~ 0
+ROW0
+Text GLabel 4600 3300 2    50   Input ~ 0
+ROW1
+Text GLabel 4600 3200 2    50   Input ~ 0
+COL0
+Text GLabel 4600 3100 2    50   Input ~ 0
+COL1
+Wire Wire Line
+	4100 2400 4000 2400
+Connection ~ 4000 2400
+Wire Wire Line
+	4000 6000 3900 6000
+Connection ~ 3900 6000
+Wire Wire Line
+	2900 3100 3050 3100
+Wire Wire Line
+	2650 3100 2800 3100
+Wire Wire Line
+	2800 3300 2450 3300
+Wire Wire Line
+	2800 3100 2800 3250
+Wire Wire Line
+	2800 3100 2900 3100
+Wire Wire Line
+	2800 3000 2800 3100
+Wire Wire Line
+	2800 3250 3050 3250
+Connection ~ 2800 3250
+Wire Wire Line
+	2800 3250 2800 3300
+Wire Wire Line
+	3050 3100 3400 3100
+Wire Wire Line
+	3050 3000 3050 3250
+Wire Wire Line
+	2450 3300 2450 3200
+Connection ~ 2450 3300
+Wire Wire Line
+	2450 3200 2450 2750
+Connection ~ 2450 3200
+Wire Wire Line
+	2650 2750 2650 2900
+Wire Wire Line
+	2650 2900 2900 2900
+Connection ~ 2900 2900
 $EndSCHEMATC
